File: schematics-kicad/schematics-kicad.kicad_sch (KiCad schematic)
At the start: 13 parts, among them U1 4051

Commit message: almost done all
Parts:
- R1, R2, R3, R4, R5: value 50K -> 100K
Changed lines of the file:
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@@
 			)
 		)
-		(property "Value" "50K"
+		(property "Value" "100K"
 			(at 236.22 43.1799 0)
 			(effects
@@
 			)
 		)
-		(property "Value" "50K"
+		(property "Value" "100K"
 			(at 220.98 43.1799 0)
 			(effects
@@
 			)
 		)
-		(property "Value" "50K"
+		(property "Value" "100K"
 			(at 278.13 43.1799 0)
 			(effects
@@
 			)
 		)
-		(property "Value" "50K"
+		(property "Value" "100K"
 			(at 251.46 43.1799 0)
 			(effects
@@
 			)
 		)
-		(property "Value" "50K"
+		(property "Value" "100K"
 			(at 265.43 43.1799 0)
 			(effects
